File: herringbone.kicad_pcb (KiCad board)
At the start: 2 copper layers, 114.3 x 122.8 mm, 91 parts, among them U1 ATmega328P-PU, Y1 16MHz

Commit message: Cleanups
Routing:
- net GND: track 211.4 -> 208.3 mm, vias 3 -> 2
- net +5V: track 165.3 -> 167.0 mm, vias 4 -> 3
- net i2c_SDA: track 119.0 -> 120.8 mm
- net Net-(F1-Pad1): track 18.4 -> 17.5 mm
- net Net-(USB1-CC2): track 17.4 -> 16.6 mm
- net Net-(D51-K): track 22.8 -> 23.5 mm
- net COL0: track 304.0 -> 303.4 mm

Commit message: Add plate and bottom.
Parts:
- added H8: M2, MountingHole:MountingHole_2.2mm_M2_Pad, F.Cu at (161.9, 85.7)
- added H9: M2, MountingHole:MountingHole_2.2mm_M2_Pad, F.Cu at (85.7, 85.7)
- S0_0, S0_1, S0_2, S0_3, S0_4, S1_0, S1_1, S1_2, S1_3, S1_4, S2_0, S2_1, S2_2, S2_3, S2_4, S3_0, S3_1, S3_2, S3_3, S3_4, S4_0, S4_1, S4_2, S4_3, S4_4, S5_0, S5_1, S5_2, S5_3, S5_4: footprint ScottoKeebs_Hotswap:Hotswap_MX_1.00u -> herringbone:Hotswap_MX_Plated_1.00u
- U1: footprint herringbone:DIP-28_W7.62mm_Socket -> herringbone:ATMEGA328-PU_DIP-28_W7.62mm_Socket
Routing:
- net COL4: track 209.8 -> 216.9 mm
- net COL3: track 262.7 -> 269.7 mm
- net COL2: track 280.1 -> 287.0 mm
- net COL0: track 303.4 -> 310.1 mm
- net COL1: track 300.2 -> 306.6 mm
- net COL5: track 113.6 -> 117.3 mm
- net Net-(D0_2-A): track 50.1 -> 53.6 mm
- net Net-(D0_4-A): track 84.3 -> 87.5 mm
- net Net-(D0_3-A): track 67.2 -> 70.3 mm
- net Net-(D0_1-A): track 33.7 -> 34.7 mm
Other:
- board text added: "Herringbone Rev1"
