File: pcb/herringbone.kicad_pcb (KiCad board)
At the start: 2 copper layers, 114.3 x 122.8 mm, 95 parts, among them U1 ATmega328P-PU, Y1 16MHz

Commit message: PCB rev2.
- Add LEDs
- Fix D+ D- USB pins for USBaspLoader to be happy
- Widen power Lines
- Allow for 2U keys in bottom corners
Parts:
- added L0: LED, LED_THT:LED_D3.0mm, F.Cu at (92.2, 42.2)
- added L1: LED, LED_THT:LED_D3.0mm, F.Cu at (92.2, 46.7)
- added R10: 5.1k, herringbone:R_Axial_DIN0204_L3.6mm_D1.6mm_P5.08mm_Horizontal, F.Cu at (79.5, 52.4)
- added R9: 5.1k, herringbone:R_Axial_DIN0204_L3.6mm_D1.6mm_P5.08mm_Horizontal, F.Cu at (79.5, 54.7)
- moved F1 2.37 mm to (108.8, 45.0)
- moved C3 1.50 mm to (88.2, 45.3)
Connections:
- B2 pad 1: Net-(U1-PD0) -> ROW0
- U1 pad 2: Net-(U1-PD0) -> ROW0
- U1 pad 26: unconnected-(U1-PC3-Pad26) -> LED0
- U1 pad 3: USB_D+ -> LED1
- U1 pad 4: USB_D- -> USB_D+
- U1 pad 5: ROW0 -> USB_D-
Routing:
- net Net-(U1-PD0): track 47.6 -> 0.00 mm, vias 2 -> 0
- net ROW0: track 68.1 -> 113.9 mm, vias 0 -> 2
- net LED1: track 0.00 -> 44.0 mm, vias 0 -> 2
- net LED0: track 0.00 -> 37.4 mm
- net Net-(L0-K): track 0.00 -> 16.2 mm
- net Net-(D50-K): track 29.5 -> 44.6 mm
- net Net-(L1-K): track 0.00 -> 9.87 mm
- net +5V: track 167.0 -> 174.6 mm, vias 3 -> 5
- net USB_D+: track 8.74 -> 13.5 mm, vias 0 -> 1
- net USB_D-: track 12.2 -> 16.8 mm, vias 0 -> 1
- net i2c_SCL: track 122.2 -> 125.0 mm, vias 2 -> 1
- net i2c_SDA: track 120.8 -> 118.9 mm
- net GND: track 208.3 -> 206.7 mm
- net ROW1: track 69.6 -> 69.0 mm

Commit message: pcb and footprint updates.
Connections:
- B2 pad 1: ROW0 -> GND
- B2 pad 2: GND -> ROW0
